Commit message: base_link and base_footprint are now defined outside of zuuu_description.urdf

File: zuuu_description/urdf/zuuu_description.urdf.xacro (robot description, xacro)
@@ -36,36 +36,4 @@
       </inertial>
     </xacro:macro>
-    <!-- Robot Footprint -->
-    <link name="base_footprint" />
-    <joint name="base_footprint_joint" type="fixed">
-      <origin rpy="0 0 0" xyz="0 0 0" />
-      <axis xyz="0 0 ${(base_top_height-base_depth/2)}" />
-      <!-- <joint_properties damping="${global_damping}" friction="${global_friction}"/> -->
-      <parent link="base_footprint" />
-      <child link="base_link" />
-    </joint>
-    <!-- Robot Base -->
-    <link name="base_link">
-      <!-- <visual>
-        <geometry>
-          <cylinder radius="${base_radius}" length="${base_depth}"/>
-        </geometry>
-        <material name="Cyan">
-          <color rgba="0 1.0 1.0 1.0"/>
-        </material>
-      </visual> -->
-      <visual>
-        <origin xyz="0 0 ${(-base_top_height+base_depth/2)}" rpy="0 0 0" />
-        <geometry>
-          <mesh filename="file://$(find zuuu_description)/meshes/reachy_mobile_pauvre.dae" />
-        </geometry>
-      </visual>
-      <collision>
-        <geometry>
-          <cylinder radius="${base_radius}" length="${base_depth}" />
-        </geometry>
-      </collision>
-      <xacro:cylinder_inertia m="20" r="${base_radius}" h="${base_depth}" />
-    </link>
     <!-- Wheels -->
     <xacro:macro name="wheel" params="prefix yaw_angle">

Commit message: fixed mobile base collisions

File: zuuu_description/urdf/zuuu_description.urdf.xacro (robot description, xacro)
@@ -59,7 +59,5 @@
           <parent link="base_link" />
           <child link="${prefix}_link" />
-          <origin
-            xyz="${wheel_radial_dist*cos(yaw_angle)} ${-wheel_radial_dist*sin(yaw_angle)} ${-((base_top_height-base_depth/2)- wheel_radius)}"
-            rpy="0 0 ${pi/2-yaw_angle}" />
+          <origin xyz="${(wheel_radial_dist+wheel_width/2)*cos(yaw_angle)} ${-(wheel_radial_dist+wheel_width/2)*sin(yaw_angle)} ${(wheel_radius)}" rpy="0 0 ${pi/2-yaw_angle}"/>
           <axis xyz="0 1 0" />
           <joint_properties damping="${global_damping}" friction="${global_friction}" />
@@ -87,5 +85,5 @@
           <joint_properties damping="${global_damping}" friction="${global_friction}" />
         </joint>
-        <!-- Physics because we're smart and handsome -->
+        <!-- Physics stuff -->
         <gazebo reference="${prefix}_link">
           <mu1 value="1.0" />
@@ -119,4 +117,35 @@
     <xacro:wheel prefix="drivewhl2" yaw_angle="${5*pi/3}" />
     <xacro:wheel prefix="drivewhl3" yaw_angle="${pi}" />
+    <!-- Robot Footprint. The robot's root link -->
+    <link name="base_footprint"/>
+    <joint name="base_footprint_joint" type="fixed">
+      <origin rpy="0 0 0" xyz="0 0 0"/>
+      <axis xyz="0 0 ${(base_top_height-base_depth/2)}"/>
+      <!-- <joint_properties damping="${global_damping}" friction="${global_friction}"/> -->
+      <parent link="base_footprint"/>
+      <child link="base_link"/>
+    </joint>
+    <link name="base_link">
+      <visual>
+        <origin xyz="0 0 0" rpy="0 0 0"/>
+        <geometry>
+          <mesh filename="file://$(find reachy_description)/meshes/mobile_base_visual.dae" />
+        </geometry>
+        <xacro:reachy_grey/>
+      </visual>
+      <collision>
+        <origin xyz="0 0 0.145" rpy="0 0 0"/>
+        <geometry>
+          <cylinder radius="0.245" length="0.19"/>
+        </geometry>
+      </collision>
+      <inertial>
+          <origin xyz="0.008 -0.00048 0.112" rpy="0 0 0"/>
+          <mass value="24.0"/>
+          <inertia ixx="0.40791094" ixy="-0.00167148" ixz="-0.00178789"
+             iyx="-0.00167148" iyy="0.4236827" iyz="0.00026596"
+             izx="-0.00178789" izy="0.00026596" izz="0.70990763"/>
+      </inertial>
+    </link>
     <link name="lidar_link">
       <inertial>
@@ -142,8 +171,8 @@
       <child link="lidar_link" />
       <!-- <origin xyz="0.155 0 0.2" rpy="0 0 0"/> -->
-      <!-- The -0.0129 were added on 22 pril 2022 for the second version of Zuuu. The 2mm pads are
+      <!-- The -0.0129 were added on 22 April 2022 for the second version of Zuuu. The 2mm pads are
       not taken into account -->
-      <origin xyz="0.155 0 ${-(base_top_height-base_depth/2)+base_top_height+0.105 -0.0129}"
-        rpy="0 0 0" />
+      <!-- <origin xyz="0.155 0 ${-(base_top_height-base_depth/2)+base_top_height+0.105 -0.0129}" rpy="0 0 0" /> -->
+      <origin xyz="0.184 0 0.25" rpy="0 0 0"/>
     </joint>
   </xacro:macro>

Commit message: Fixing mobile base slides on gazebo

File: zuuu_description/urdf/zuuu_description.urdf.xacro (robot description, xacro)
@@ -134,8 +134,16 @@
         <xacro:reachy_grey/>
       </visual>
-      <collision>
+      <!-- Real collision -->
+      <!-- <collision>
         <origin xyz="0 0 0.145" rpy="0 0 0"/>
         <geometry>
           <cylinder radius="0.245" length="0.19"/>
+        </geometry>
+      </collision> -->
+      <!-- exagerated collision to avoid the mobile base sliding on Gazebo -->
+      <collision>
+        <origin xyz="0 0 0.12" rpy="0 0 0"/>
+        <geometry>
+          <cylinder radius="0.245" length="0.24"/>
         </geometry>
       </collision>

Commit message: Fixing robot falls or robot slides in Gazebo. Wheels collide on the floor with friction now

File: zuuu_description/urdf/zuuu_description.urdf.xacro (robot description, xacro)
@@ -56,4 +56,5 @@
       </link>
       <xacro:if value="$(arg use_fixed_wheels)">
+        <!-- If use_fixed_wheels the wheels can't rotate, they will slide on the floor -->
         <joint name="${prefix}_joint" type="fixed">
           <parent link="base_link" />
@@ -63,8 +64,7 @@
           <joint_properties damping="${global_damping}" friction="${global_friction}" />
         </joint>
-        <!-- No friction because we suck and everything is lame -->
         <gazebo reference="${prefix}_link">
-          <mu1 value="0.0" />
-          <mu2 value="0.0" />
+          <mu1 value="0.1" />
+          <mu2 value="0.1" />
           <kp value="10000000.0" />
           <kd value="1.0" />
@@ -76,4 +76,5 @@
       </xacro:if>
       <xacro:unless value="$(arg use_fixed_wheels)">
+        <!-- If not use_fixed_wheels the wheels will rotate. The friction parameters try to emulate holonomic wheels, it kinda works but is unreliable with Gazebo -->
         <joint name="${prefix}_joint" type="continuous">
           <parent link="base_link" />
@@ -135,17 +136,17 @@
       </visual>
       <!-- Real collision -->
-      <!-- <collision>
+      <collision>
         <origin xyz="0 0 0.145" rpy="0 0 0"/>
         <geometry>
           <cylinder radius="0.245" length="0.19"/>
         </geometry>
-      </collision> -->
+      </collision>
       <!-- exagerated collision to avoid the mobile base sliding on Gazebo -->
-      <collision>
+      <!-- <collision>
         <origin xyz="0 0 0.12" rpy="0 0 0"/>
         <geometry>
           <cylinder radius="0.245" length="0.24"/>
         </geometry>
-      </collision>
+      </collision> -->
       <inertial>
           <origin xyz="0.008 -0.00048 0.112" rpy="0 0 0"/>

Commit message: LIDAR filter and safety now works in gazebo mode

File: zuuu_description/urdf/zuuu_description.urdf.xacro (robot description, xacro)
@@ -183,5 +183,5 @@
       not taken into account -->
       <!-- <origin xyz="0.155 0 ${-(base_top_height-base_depth/2)+base_top_height+0.105 -0.0129}" rpy="0 0 0" /> -->
-      <origin xyz="0.184 0 0.25" rpy="0 0 0"/>
+      <origin xyz="0.184 0 0.25" rpy="0 0 3.141592653589793"/>
     </joint>
   </xacro:macro>
