Commit message: created a zuuu_nav2_config folder and re-rganized

File: zuuu_description/urdf/zuuu.gazebo.xacro (robot description, xacro)
@@ -1,164 +1,60 @@
 <?xml version="1.0"?>
 <robot xmlns:xacro="http://ros.org/wiki/xacro">
-  <xacro:macro name="zuuu_gazebo" params="model prefix">
-    <gazebo>
-        <plugin name="object_controller" filename="libgazebo_ros_planar_move.so">
-        <commandTopic>cmd_vel</commandTopic>
-        <odometryTopic>odom</odometryTopic>
-        <robotNamespace> </robotNamespace>
-        <!-- Set control loop update rate -->
-        <odometryRate>100</odometryRate>
-        <!-- Set odom publish rate -->
-        <publish_rate>100</publish_rate>
-        <!-- Set if odom required -->
-        <publish_odom>true</publish_odom>
-        <publish_odom_tf>true</publish_odom_tf>
-        <!-- Frame IDs -->
-        <odometryFrame>odom</odometryFrame>
-        <robotBaseFrame>base_link</robotBaseFrame>
-        <!-- Set odom covariance -->
-        <covariance_x>0.0001</covariance_x>
-        <covariance_y>0.0001</covariance_y>
-        <covariance_yaw>0.01</covariance_yaw>
-        </plugin>
-    </gazebo>
-    <gazebo reference="imu_link">
-        <sensor name="imu_sensor" type="imu">
-        <plugin filename="libgazebo_ros_imu_sensor.so" name="imu_plugin">
-            <ros>
-            <namespace></namespace>
-            <remapping>~/out:=imu</remapping>
-            </ros>
-            <initial_orientation_as_reference>false</initial_orientation_as_reference>
-        </plugin>
-        <always_on>true</always_on>
-        <update_rate>100</update_rate>
-        <visualize>true</visualize>
-        <imu>
-            <angular_velocity>
-            <x>
-                <noise type="gaussian">
-                <mean>0.0</mean>
-                <stddev>2e-4</stddev>
-                <bias_mean>0.0000075</bias_mean>
-                <bias_stddev>0.0000008</bias_stddev>
-                </noise>
-            </x>
-            <y>
-                <noise type="gaussian">
-                <mean>0.0</mean>
-                <stddev>2e-4</stddev>
-                <bias_mean>0.0000075</bias_mean>
-                <bias_stddev>0.0000008</bias_stddev>
-                </noise>
-            </y>
-            <z>
-                <noise type="gaussian">
-                <mean>0.0</mean>
-                <stddev>2e-4</stddev>
-                <bias_mean>0.0000075</bias_mean>
-                <bias_stddev>0.0000008</bias_stddev>
-                </noise>
-            </z>
-            </angular_velocity>
-            <linear_acceleration>
-            <x>
-                <noise type="gaussian">
-                <mean>0.0</mean>
-                <stddev>1.7e-2</stddev>
-                <bias_mean>0.1</bias_mean>
-                <bias_stddev>0.001</bias_stddev>
-                </noise>
-            </x>
-            <y>
-                <noise type="gaussian">
-                <mean>0.0</mean>
-                <stddev>1.7e-2</stddev>
-                <bias_mean>0.1</bias_mean>
-                <bias_stddev>0.001</bias_stddev>
-                </noise>
-            </y>
-            <z>
-                <noise type="gaussian">
-                <mean>0.0</mean>
-                <stddev>1.7e-2</stddev>
-                <bias_mean>0.1</bias_mean>
-                <bias_stddev>0.001</bias_stddev>
-                </noise>
-            </z>
-            </linear_acceleration>
-        </imu>
-        </sensor>
-    </gazebo>
-    <gazebo reference="lidar_link">
-        <sensor name="lidar" type="ray">
-        <always_on>true</always_on>
-        <visualize>true</visualize>
-        <update_rate>5</update_rate>
-        <ray>
-            <scan>
-            <horizontal>
-                <samples>360</samples>
-                <resolution>1.000000</resolution>
-                <min_angle>0.000000</min_angle>
-                <max_angle>6.280000</max_angle>
-            </horizontal>
-            </scan>
-            <range>
-            <min>0.120000</min>
-            <max>20</max>
-            <resolution>0.015000</resolution>
-            </range>
-            <noise>
-            <type>gaussian</type>
-            <mean>0.0</mean>
-            <stddev>0.01</stddev>
-            </noise>
-        </ray>
-        <plugin name="scan" filename="libgazebo_ros_ray_sensor.so">
-            <ros>
-            <remapping>~/out:=scan</remapping>
-            </ros>
-            <output_type>sensor_msgs/LaserScan</output_type>
-            <frame_name>lidar_link</frame_name>
-        </plugin>
-        </sensor>
-    </gazebo>
-    <gazebo reference="camera_link">
-        <sensor name="depth_camera" type="depth">
-        <visualize>true</visualize>
-        <update_rate>30.0</update_rate>
-        <camera name="camera">
-            <horizontal_fov>1.047198</horizontal_fov>
-            <image>
-            <width>640</width>
-            <height>480</height>
-            <format>R8G8B8</format>
-            </image>
-            <clip>
-            <near>0.05</near>
-            <far>3</far>
-            </clip>
-        </camera>
-        <plugin name="depth_camera_controller" filename="libgazebo_ros_camera.so">
-            <baseline>0.2</baseline>
-            <alwaysOn>true</alwaysOn>
-            <updateRate>0.0</updateRate>
-            <frame_name>camera_depth_frame</frame_name>
-            <pointCloudCutoff>0.5</pointCloudCutoff>
-            <pointCloudCutoffMax>3.0</pointCloudCutoffMax>
-            <distortionK1>0</distortionK1>
-            <distortionK2>0</distortionK2>
-            <distortionK3>0</distortionK3>
-            <distortionT1>0</distortionT1>
-            <distortionT2>0</distortionT2>
-            <CxPrime>0</CxPrime>
-            <Cx>0</Cx>
-            <Cy>0</Cy>
-            <focalLength>0</focalLength>
-            <hackBaseline>0</hackBaseline>
-        </plugin>
-        </sensor>
-    </gazebo>
-  </xacro:macro>
+    <xacro:macro name="zuuu_gazebo" params="model prefix">
+        <gazebo>
+            <plugin name="object_controller" filename="libgazebo_ros_planar_move.so">
+                <commandTopic>cmd_vel</commandTopic>
+                <odometryTopic>odom</odometryTopic>
+                <robotNamespace> </robotNamespace>
+                <!-- Set control loop update rate -->
+                <odometryRate>100</odometryRate>
+                <!-- Set odom publish rate -->
+                <publish_rate>100</publish_rate>
+                <!-- Set if odom required -->
+                <publish_odom>true</publish_odom>
+                <publish_odom_tf>true</publish_odom_tf>
+                <!-- Frame IDs -->
+                <odometryFrame>odom</odometryFrame>
+                <robotBaseFrame>base_link</robotBaseFrame>
+                <!-- Set odom covariance -->
+                <covariance_x>0.0001</covariance_x>
+                <covariance_y>0.0001</covariance_y>
+                <covariance_yaw>0.01</covariance_yaw>
+            </plugin>
+        </gazebo>
+        <gazebo reference="lidar_link">
+            <sensor name="lidar" type="ray">
+                <always_on>true</always_on>
+                <visualize>true</visualize>
+                <update_rate>5</update_rate>
+                <ray>
+                    <scan>
+                        <horizontal>
+                            <samples>360</samples>
+                            <resolution>1.000000</resolution>
+                            <min_angle>0.000000</min_angle>
+                            <max_angle>6.280000</max_angle>
+                        </horizontal>
+                    </scan>
+                    <range>
+                        <min>0.120000</min>
+                        <max>20</max>
+                        <resolution>0.015000</resolution>
+                    </range>
+                    <noise>
+                        <type>gaussian</type>
+                        <mean>0.0</mean>
+                        <stddev>0.01</stddev>
+                    </noise>
+                </ray>
+                <plugin name="scan" filename="libgazebo_ros_ray_sensor.so">
+                    <ros>
+                        <remapping>~/out:=scan</remapping>
+                    </ros>
+                    <output_type>sensor_msgs/LaserScan</output_type>
+                    <frame_name>lidar_link</frame_name>
+                </plugin>
+            </sensor>
+        </gazebo>
+    </xacro:macro>
 </robot>

File: zuuu_description/urdf/zuuu.urdf.xacro (robot description, xacro)
@@ -1,16 +1,16 @@
 <?xml version="1.0"?>
 <robot xmlns:xacro="http://www.ros.org/wiki/xacro" name="zuuu">
-  <xacro:arg name="prefix" default=""/>
+  <xacro:arg name="prefix" default="" />
   <xacro:arg name="model" default="" />
-  <xacro:arg name="use_gazebo" default="true"/>
-  <xacro:arg name="use_fake_components" default="true"/>
-  <xacro:arg name="use_fixed_wheels" default="true"/>
-  <xacro:arg name="use_ros_control" default="true"/>
+  <xacro:arg name="use_gazebo" default="true" />
+  <xacro:arg name="use_fake_components" default="true" />
+  <xacro:arg name="use_fixed_wheels" default="true" />
+  <xacro:arg name="use_ros_control" default="true" />
   <!-- Import zuuu macro -->
-  <xacro:include filename="$(find zuuu_description)/urdf/zuuu_description.urdf.xacro"/>
+  <xacro:include filename="$(find zuuu_description)/urdf/zuuu_description.urdf.xacro" />
   <!-- Import Gazebo macro -->
-  <xacro:include filename="$(find zuuu_description)/urdf/zuuu.gazebo.xacro"/>
+  <xacro:include filename="$(find zuuu_description)/urdf/zuuu.gazebo.xacro" />
   <!-- Import Zuuu ros2_control description -->
-  <xacro:include filename="$(find zuuu_description)/urdf/zuuu.ros2_control.xacro"/>
+  <xacro:include filename="$(find zuuu_description)/urdf/zuuu.ros2_control.xacro" />
   <xacro:zuuu
     model="$(arg model)" prefix="$(arg prefix)">
@@ -20,5 +20,5 @@
   </xacro:if>
   <xacro:if value="$(arg use_ros_control)">
-    <xacro:zuuu_ros2_control model="$(arg model)" prefix="$(arg prefix)"/>
+    <xacro:zuuu_ros2_control model="$(arg model)" prefix="$(arg prefix)" />
   </xacro:if>
 </robot>

File: zuuu_description/urdf/zuuu_description.urdf.xacro (robot description, xacro)
@@ -3,19 +3,20 @@
   <xacro:macro name="zuuu" params="model prefix">
     <!-- Define robot constants -->
-    <xacro:property name="base_radius" value="0.16"/>
-    <xacro:property name="base_top_height" value="0.1425"/>
-    <xacro:property name="base_depth" value="0.07"/>
-    <xacro:property name="wheel_radius" value="0.105"/>
-    <xacro:property name="wheel_width" value="0.035"/>
-    <xacro:property name="wheel_radial_dist" value="0.1805"/>
-    <xacro:property name="wheel_zoff" value="0.20"/>
-    <xacro:property name="global_damping" value="0.5"/>
-    <xacro:property name="global_friction" value="0.1"/>
+    <xacro:property name="base_radius" value="0.16" />
+    <xacro:property name="base_top_height" value="0.1425" />
+    <xacro:property name="base_depth" value="0.07" />
+    <xacro:property name="wheel_radius" value="0.105" />
+    <xacro:property name="wheel_width" value="0.035" />
+    <xacro:property name="wheel_radial_dist" value="0.1805" />
+    <xacro:property name="wheel_zoff" value="0.20" />
+    <xacro:property name="global_damping" value="0.5" />
+    <xacro:property name="global_friction" value="0.1" />
     <!-- Define some commonly used intertial properties  -->
     <xacro:macro name="box_inertia" params="m w h d">
       <inertial>
-        <origin xyz="0 0 0" rpy="${pi/2} 0 ${pi/2}"/>
-        <mass value="${m}"/>
-        <inertia ixx="${(m/12) * (h*h + d*d)}" ixy="0.0" ixz="0.0" iyy="${(m/12) * (w*w + d*d)}" iyz="0.0" izz="${(m/12) * (w*w + h*h)}"/>
+        <origin xyz="0 0 0" rpy="${pi/2} 0 ${pi/2}" />
+        <mass value="${m}" />
+        <inertia ixx="${(m/12) * (h*h + d*d)}" ixy="0.0" ixz="0.0" iyy="${(m/12) * (w*w + d*d)}"
+          iyz="0.0" izz="${(m/12) * (w*w + h*h)}" />
       </inertial>
     </xacro:macro>
@@ -23,22 +24,24 @@
       <inertial>
         <origin xyz="0 0 0" rpy="${pi/2} 0 0" />
-        <mass value="${m}"/>
-        <inertia ixx="${(m/12) * (3*r*r + h*h)}" ixy = "0" ixz = "0" iyy="${(m/12) * (3*r*r + h*h)}" iyz = "0" izz="${(m/2) * (r*r)}"/>
+        <mass value="${m}" />
+        <inertia ixx="${(m/12) * (3*r*r + h*h)}" ixy="0" ixz="0" iyy="${(m/12) * (3*r*r + h*h)}"
+          iyz="0" izz="${(m/2) * (r*r)}" />
       </inertial>
     </xacro:macro>
     <xacro:macro name="sphere_inertia" params="m r">
       <inertial>
-        <mass value="${m}"/>
-        <inertia ixx="${(2/5) * m * (r*r)}" ixy="0.0" ixz="0.0" iyy="${(2/5) * m * (r*r)}" iyz="0.0" izz="${(2/5) * m * (r*r)}"/>
+        <mass value="${m}" />
+        <inertia ixx="${(2/5) * m * (r*r)}" ixy="0.0" ixz="0.0" iyy="${(2/5) * m * (r*r)}" iyz="0.0"
+          izz="${(2/5) * m * (r*r)}" />
       </inertial>
     </xacro:macro>
     <!-- Robot Footprint -->
-    <link name="base_footprint"/>
+    <link name="base_footprint" />
     <joint name="base_footprint_joint" type="fixed">
-      <origin rpy="0 0 0" xyz="0 0 0"/>
-      <axis xyz="0 0 ${(base_top_height-base_depth/2)}"/>
+      <origin rpy="0 0 0" xyz="0 0 0" />
+      <axis xyz="0 0 ${(base_top_height-base_depth/2)}" />
       <!-- <joint_properties damping="${global_damping}" friction="${global_friction}"/> -->
-      <parent link="base_footprint"/>
-      <child link="base_link"/>
+      <parent link="base_footprint" />
+      <child link="base_link" />
     </joint>
     <!-- Robot Base -->
@@ -53,15 +56,15 @@
       </visual> -->
       <visual>
-        <origin xyz="0 0 ${(-base_top_height+base_depth/2)}" rpy="0 0 0"/>
+        <origin xyz="0 0 ${(-base_top_height+base_depth/2)}" rpy="0 0 0" />
         <geometry>
-          <mesh filename="file://$(find zuuu_description)/meshes/reachy_mobile_pauvre.dae"/>
+          <mesh filename="file://$(find zuuu_description)/meshes/reachy_mobile_pauvre.dae" />
         </geometry>
       </visual>
       <collision>
         <geometry>
-          <cylinder radius="${base_radius}" length="${base_depth}"/>
+          <cylinder radius="${base_radius}" length="${base_depth}" />
         </geometry>
       </collision>
-      <xacro:cylinder_inertia m="20" r="${base_radius}" h="${base_depth}"/>
+      <xacro:cylinder_inertia m="20" r="${base_radius}" h="${base_depth}" />
     </link>
     <!-- Wheels -->
@@ -77,46 +80,50 @@
         </visual> -->
         <collision>
-          <origin xyz="0 0 0" rpy="${pi/2} 0 0"/>
+          <origin xyz="0 0 0" rpy="${pi/2} 0 0" />
           <geometry>
-            <cylinder radius="${wheel_radius}" length="${wheel_width}"/>
+            <cylinder radius="${wheel_radius}" length="${wheel_width}" />
           </geometry>
         </collision>
-        <xacro:cylinder_inertia m="0.5" r="${wheel_radius}" h="${wheel_width}"/>
+        <xacro:cylinder_inertia m="0.5" r="${wheel_radius}" h="${wheel_width}" />
       </link>
       <xacro:if value="$(arg use_fixed_wheels)">
-          <joint name="${prefix}_joint" type="fixed">
-            <parent link="base_link"/>
-            <child link="${prefix}_link"/>
-            <origin xyz="${wheel_radial_dist*cos(yaw_angle)} ${-wheel_radial_dist*sin(yaw_angle)} ${-((base_top_height-base_depth/2)- wheel_radius)}" rpy="0 0 ${pi/2-yaw_angle}"/>
-            <axis xyz="0 1 0"/>
-            <joint_properties damping="${global_damping}" friction="${global_friction}"/>
-          </joint>
-          <!-- No friction because we suck and everything is lame -->
-          <gazebo reference="${prefix}_link">
-            <mu1 value="0.0"/>
-            <mu2 value="0.0"/>
-            <kp value="10000000.0" />
-            <kd value="1.0" />
-            <fdir1 value="1 0 0"/>
-            <maxVel>1.0</maxVel>
-            <minDepth>0.0</minDepth>
-            <turnGravityOff>false</turnGravityOff>
-          </gazebo>
+        <joint name="${prefix}_joint" type="fixed">
+          <parent link="base_link" />
+          <child link="${prefix}_link" />
+          <origin
+            xyz="${wheel_radial_dist*cos(yaw_angle)} ${-wheel_radial_dist*sin(yaw_angle)} ${-((base_top_height-base_depth/2)- wheel_radius)}"
+            rpy="0 0 ${pi/2-yaw_angle}" />
+          <axis xyz="0 1 0" />
+          <joint_properties damping="${global_damping}" friction="${global_friction}" />
+        </joint>
+        <!-- No friction because we suck and everything is lame -->
+        <gazebo reference="${prefix}_link">
+          <mu1 value="0.0" />
+          <mu2 value="0.0" />
+          <kp value="10000000.0" />
+          <kd value="1.0" />
+          <fdir1 value="1 0 0" />
+          <maxVel>1.0</maxVel>
+          <minDepth>0.0</minDepth>
+          <turnGravityOff>false</turnGravityOff>
+        </gazebo>
       </xacro:if>
       <xacro:unless value="$(arg use_fixed_wheels)">
         <joint name="${prefix}_joint" type="continuous">
-          <parent link="base_link"/>
-          <child link="${prefix}_link"/>
-          <origin xyz="${wheel_radial_dist*cos(yaw_angle)} ${-wheel_radial_dist*sin(yaw_angle)} ${-((base_top_height-base_depth/2)- wheel_radius)}" rpy="0 0 ${pi/2-yaw_angle}"/>
-          <axis xyz="0 1 0"/>
-          <joint_properties damping="${global_damping}" friction="${global_friction}"/>
+          <parent link="base_link" />
+          <child link="${prefix}_link" />
+          <origin
+            xyz="${wheel_radial_dist*cos(yaw_angle)} ${-wheel_radial_dist*sin(yaw_angle)} ${-((base_top_height-base_depth/2)- wheel_radius)}"
+            rpy="0 0 ${pi/2-yaw_angle}" />
+          <axis xyz="0 1 0" />
+          <joint_properties damping="${global_damping}" friction="${global_friction}" />
         </joint>
         <!-- Physics because we're smart and handsome -->
         <gazebo reference="${prefix}_link">
-          <mu1 value="1.0"/>
-          <mu2 value="0.0"/>
+          <mu1 value="1.0" />
+          <mu2 value="0.0" />
           <kp value="10000000.0" />
           <kd value="1.0" />
-          <fdir1 value="1 0 0"/>
+          <fdir1 value="1 0 0" />
           <maxVel>5.0</maxVel>
           <minDepth>0.002</minDepth>
@@ -134,8 +141,8 @@
       </link>
       <joint name="${prefix}_extra_joint" type="fixed">
-        <origin rpy="0 0 0" xyz="0 0 0"/>
-        <axis xyz="0 0 0"/>
-        <parent link="${prefix}_link"/>
-        <child link="${prefix}_extra_link"/>
+        <origin rpy="0 0 0" xyz="0 0 0" />
+        <axis xyz="0 0 0" />
+        <parent link="${prefix}_link" />
+        <child link="${prefix}_extra_link" />
       </joint>
     </xacro:macro>
@@ -144,32 +151,14 @@
     <xacro:wheel prefix="drivewhl2" yaw_angle="${5*pi/3}" />
     <xacro:wheel prefix="drivewhl3" yaw_angle="${pi}" />
-    <link name="imu_link">
-      <!-- <visual>
-        <geometry>
-          <box size="0.1 0.1 0.02"/>
-        </geometry>
-      </visual> -->
-      <collision>
-        <geometry>
-          <box size="0.1 0.1 0.1"/>
-        </geometry>
-      </collision>
-      <xacro:box_inertia m="0.1" w="0.1" d="0.1" h="0.1"/>
-    </link>
-    <joint name="imu_joint" type="fixed">
-      <parent link="base_link"/>
-      <child link="imu_link"/>
-      <origin xyz="0 0 0.01"/>
-    </joint>
     <link name="lidar_link">
       <inertial>
-        <origin xyz="0 0 0" rpy="0 0 0"/>
-        <mass value="0.125"/>
-        <inertia ixx="0.001"  ixy="0"  ixz="0" iyy="0.001" iyz="0" izz="0.001" />
+        <origin xyz="0 0 0" rpy="0 0 0" />
+        <mass value="0.125" />
+        <inertia ixx="0.001" ixy="0" ixz="0" iyy="0.001" iyz="0" izz="0.001" />
       </inertial>
       <collision>
-        <origin xyz="0 0 0" rpy="0 0 0"/>
+        <origin xyz="0 0 0" rpy="0 0 0" />
         <geometry>
-          <cylinder radius="0.0508" length="0.055"/>
+          <cylinder radius="0.0508" length="0.055" />
         </geometry>
       </collision>
@@ -182,39 +171,11 @@
     </link>
     <joint name="lidar_joint" type="fixed">
-      <parent link="base_link"/>
-      <child link="lidar_link"/>
+      <parent link="base_link" />
+      <child link="lidar_link" />
       <!-- <origin xyz="0.155 0 0.2" rpy="0 0 0"/> -->
-      <!-- The -0.0129 were added on 22 pril 2022 for the second version of Zuuu. The 2mm pads are not taken into account -->
-      <origin xyz="0.155 0 ${-(base_top_height-base_depth/2)+base_top_height+0.105 -0.0129}" rpy="0 0 0"/>
-    </joint>
-    <link name="camera_link">
-      <!-- <visual>
-        <origin xyz="0 0 0" rpy="0 0 0"/>
-        <geometry>
-          <box size="0.015 0.130 0.022"/>
-        </geometry>
-      </visual> -->
-      <collision>
-        <origin xyz="0 0 0" rpy="0 0 0"/>
-        <geometry>
-          <box size="0.015 0.130 0.022"/>
-        </geometry>
-      </collision>
-      <inertial>
-        <origin xyz="0 0 0" rpy="0 0 0"/>
-        <mass value="0.035"/>
-        <inertia ixx="0.001"  ixy="0"  ixz="0" iyy="0.001" iyz="0" izz="0.001" />
-      </inertial>
-    </link>
-    <joint name="camera_joint" type="fixed">
-      <parent link="base_link"/>
-      <child link="camera_link"/>
-      <origin xyz="0.155 0 0.5" rpy="0 0 0"/>
-    </joint>
-    <link name="camera_depth_frame"/>
-    <joint name="camera_depth_joint" type="fixed">
-      <origin xyz="0 0 0" rpy="${-pi/2} 0 ${-pi/2}"/>
-      <parent link="camera_link"/>
-      <child link="camera_depth_frame"/>
+      <!-- The -0.0129 were added on 22 pril 2022 for the second version of Zuuu. The 2mm pads are
+      not taken into account -->
+      <origin xyz="0.155 0 ${-(base_top_height-base_depth/2)+base_top_height+0.105 -0.0129}"
+        rpy="0 0 0" />
     </joint>
   </xacro:macro>
